File: Baballe/untitled.sch (EAGLE design)
At the start: 12 parts, among them Q1 MOSFET-NCHANNELBSS123LT1G, Q2 MOSFET-NCHANNELBSS123LT1G, Q3 MOSFET-NCHANNELBSS123LT1G

Commit message: Travail en cours sur la V2 de la baballe.
Parts:
- removed R7, R8, R9: (no value), SparkFun-Passives:RESISTORPTH-1/2W
- added B-ALIM: (no value), SparkFun-Connectors:M02PTH
- added B-CMD, B-LED1, B-LED2: (no value), SparkFun-Connectors:M03PTH
- added C1: (no value), SparkFun-Passives:CAP0805
- added J4, J5, J6: (no value), SparkFun-Connectors:M01PTH
- added R4, R5, R6: (no value), SparkFun-Passives:RESISTOR0805-RES
- added U$1: ESP07-16PIN, baballe-module:ESP07-16PIN
- J1: device SparkFun-Connectors:M02PTH -> SparkFun-Connectors:M01PTH
- J2, J3: device SparkFun-Connectors:M03PTH -> SparkFun-Connectors:M01PTH
Connections:
- new net B-BLUE: U$1.GPIO16
- new net N$4: R6.2, U$1.CH_PD
- new net N$5: R5.1, U$1.GPIO0
- new net N$6: R4.1, U$1.GPIO15
- new net SBUTTON: U$1.GPIO13
- net D-BLUE: now also B-LED1.3, B-LED2.3; no longer J2.3
- net D-GREEN: now also B-LED1.2, B-LED2.2; no longer J2.2
- net D-RED: now also B-LED1.1, B-LED2.1; no longer J2.1
- net G-BLUE: now also B-CMD.3; no longer J3.3
- net G-GREEN: now also B-CMD.2, U$1.GPIO14; no longer J3.2
- net G-RED: now also B-CMD.1, U$1.GPIO12; no longer J3.1
- net GND: now also B-ALIM.1, C1.2, R4.2, U$1.GND; no longer J1.1, R7.1, R8.1, R9.1
- net N$7: now also J1.1; no longer R7.2
- net N$8: now also J3.1; no longer R8.2
- net N$9: now also J5.1; no longer R9.2
- net VCC: now also B-ALIM.2, C1.1, R5.2, R6.1, U$1.GPIO2, U$1.VCC; no longer J1.2
