File: Luciole/Alimentation/alimentation.brd (EAGLE design)
At the start: 30.1 x 30 mm, 19 parts, among them J1 LiPo, J2 USB-MICROB, Q1 2.5A/30V, U1 MCP73831, U2 3.3V

Commit message: Luciole V1 Ok ; Baballe V1 En cours
Parts:
- moved C1 3.70 mm to (17.1, 55.9), turned to 90 degrees
Routing:
- net GND: track 14.4 -> 29.3 mm, vias 0 -> 1
- net V_BATT: track 71.6 -> 82.6 mm, vias 1 -> 3
- net VIN: track 29.5 -> 38.8 mm, vias 2 -> 3
- net VUSB: track 28.1 -> 32.5 mm

Commit message: V2 de la Baballe
Parts:
- R1: value 2K -> 4.7K
- R2: value ? -> 200
Changed lines of the file:
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@@
 <attribute name="PROD_ID" value="TRANS-11308" x="21.59" y="67.945" size="1.778" layer="27" rot="R180" display="off"/>
 </element>
-<element name="R1" library="SparkFun-Passives" package="0805" value="2K" x="17.78" y="72.39" rot="R270"/>
-<element name="R2" library="SparkFun-Passives" package="0805" value="?" x="15.24" y="72.39" rot="R270"/>
+<element name="R1" library="SparkFun-Passives" package="0805" value="4.7K" x="17.78" y="72.39" rot="R270"/>
+<element name="R2" library="SparkFun-Passives" package="0805" value="200" x="15.24" y="72.39" rot="R270"/>
 <element name="R3" library="SparkFun-Passives" package="0805" value="10K" x="20.955" y="58.42"/>
 <element name="R4" library="SparkFun-Passives" package="0805" value="200" x="8.255" y="73.66" rot="R270"/>
