File: Luciole/Alimentation/alimentation.sch (EAGLE design)
At the start: 19 parts, among them J1 LiPo, J2 USB-MICROB, Q1 2.5A/30V, U1 MCP73831, U2 3.3V

Commit message: V2 de la Baballe
Parts:
- R1: value 2K -> 4.7K
- R2: value ? -> 200
Changed lines of the file:
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@@
 <part name="U1" library="SparkFun-PowerIC" deviceset="MCP73831" device=""/>
 <part name="GND3" library="SparkFun-Aesthetics" deviceset="GND" device=""/>
-<part name="R1" library="SparkFun-Passives" deviceset="RESISTOR" device="0805-RES" value="2K"/>
+<part name="R1" library="SparkFun-Passives" deviceset="RESISTOR" device="0805-RES" value="4.7K"/>
 <part name="GND4" library="SparkFun-Aesthetics" deviceset="GND" device=""/>
 <part name="GND5" library="SparkFun-Aesthetics" deviceset="GND" device=""/>
 <part name="GND6" library="SparkFun-Aesthetics" deviceset="GND" device=""/>
-<part name="R2" library="SparkFun-Passives" deviceset="RESISTOR" device="0805-RES" value="?"/>
+<part name="R2" library="SparkFun-Passives" deviceset="RESISTOR" device="0805-RES" value="200"/>
 <part name="LED1" library="eagle-ltspice" deviceset="LED_E" device="" value="JAUNE"/>
 <part name="R3" library="SparkFun-Passives" deviceset="RESISTOR" device="0805-RES" value="10K"/>
@@
 <sheet>
 <plain>
-<text x="5.08" y="66.04" size="1.778" layer="91">Dépend de la capacité de la batterie.
+<text x="63.5" y="63.5" size="1.778" layer="91">Dépend de la capacité de la batterie.
 Le courant de charge dépend de la batterie
 et ne doit pas dépasser la capacité.</text>
